File: Project/Project 20 - Kotak Pos Pintar/Rangkaian/layout.brd (EAGLE design)
At the start: 91.1 x 64.8 mm, 18 parts, among them X1 TERMINAL-BLOCK-3.5MM-2-PIN-LO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, X2 TERMINAL-BLOCK-3.5MM-2-PIN-LO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, X3 TERMINAL-BLOCK-3.5MM-2-PIN-LO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

Commit message: update 8 mei 2024
Parts:
- moved X1 19.1 mm to (7.62, 58.4), turned to 0 degrees
- moved X3 19.1 mm to (27.9, 58.4), turned to 0 degrees
- moved STEP_DOWN1 15.2 mm to (24.1, 15.2), flipped to the bottom
- moved JP1 1.27 mm to (33.0, 21.6)
- flipped X2 to the bottom
Routing:
- net GND1: track 301.1 -> 164.7 mm
- net 5V: track 225.0 -> 175.3 mm
- net LIMITSW2: track 38.9 -> 29.2 mm
- net IN+: track 21.1 -> 11.5 mm
- net GND: track 77.7 -> 79.4 mm
- net N$2: track 5.39 -> 6.74 mm
- net N$3: track 5.39 -> 6.74 mm
- net N$9: track 8.89 -> 7.62 mm
- net N$8: track 8.89 -> 7.62 mm
- net N$7: track 8.89 -> 7.62 mm
- net N$6: track 8.89 -> 7.62 mm
- net N$5: track 8.89 -> 7.62 mm
- net N$12: track 8.89 -> 7.62 mm
- net N$11: track 8.89 -> 7.62 mm
- net N$10: track 8.89 -> 7.62 mm
